File: africube2.sch (KiCad schematic (older format))
At the start: 21 parts, among them J1 SMA Edge FM, J2 Conn_01x04, J3 RPi_GPIO, U1 TQP7M9105, U2 SXBP-150+, U3 BA178M05FP-E2

Commit message: pcb placement
Parts:
- U2: footprint (none) -> RF_Mini-Circuits:Mini-Circuits_HF1139_LandPatternPL-230
- U3: footprint (none) -> TO_SOT_Packages_SMD:TO-252-3_TabPin2
Changed lines of the file:
@@
 F 0 "U2" H 6100 1800 60  0000 C CNN
 F 1 "SXBP-150+" H 6100 2300 60  0000 C CNN
-F 2 "" H 6100 1900 60  0001 C CNN
+F 2 "RF_Mini-Circuits:Mini-Circuits_HF1139_LandPatternPL-230" H 6100 1900 60  0001 C CNN
 F 3 "" H 6100 1900 60  0001 C CNN
 	1    6100 2050
@@
 F 0 "U3" H 6300 3000 60  0000 C CNN
 F 1 "BA178M05FP-E2" H 6250 3450 60  0000 C CNN
-F 2 "" H 6200 3200 60  0001 C CNN
+F 2 "TO_SOT_Packages_SMD:TO-252-3_TabPin2" H 6200 3200 60  0001 C CNN
 F 3 "" H 6200 3200 60  0001 C CNN
 	1    6200 3150
