File: africube2.sch (KiCad schematic (older format))
At the start: 36 parts, among them IC1 ADC-20-4, J1 SMA Edge FM, J2 Conn_01x04, J3 RPi_GPIO, J4 Conn_01x02, U1 TQP7M9105, U2 SXBP-150+, U3 BA178M05FP-E2, U4 MCP3421A0T-E/CH

Commit message: removing power detector
Parts:
- D2: footprint (none) -> Diodes_SMD:D_SOD-523
- IC1: footprint ADC-20-4+ -> rf_noise:ADC-20-4+
- U3: footprint TO_SOT_Packages_SMD:TO-252-3_TabPin2 -> TO_SOT_Packages_SMD:TO-252-3_TabPin4
- U4: footprint (none) -> TO_SOT_Packages_SMD:SOT-23-6_Handsoldering
- gave numbers to parts that had none: 1
Changed lines of the file:
@@
 LIBS:contrib
 LIBS:valves
-LIBS:analog_devices
+LIBS:africube2-cache
+LIBS:vhf_uhf_IQ_Modulator_V4-cache
+LIBS:raspberrrypi_hat-cache
+LIBS:dk_RF-Amplifiers
+LIBS:africube_v1-cache
+LIBS:adc-20-4
+LIBS:HamShield09-cache
+LIBS:BA178M05FP-E2
+LIBS:ADC-20-4
+LIBS:ADC-15-4+
 LIBS:AD8317
-LIBS:ADC-15-4+
-LIBS:adc-20-4
-LIBS:africube2-cache
 EELAYER 25 0
 EELAYER END
@@
 F 0 "U3" H 6300 3000 60  0000 C CNN
 F 1 "BA178M05FP-E2" H 6250 3450 60  0000 C CNN
-F 2 "TO_SOT_Packages_SMD:TO-252-3_TabPin2" H 6200 3200 60  0001 C CNN
+F 2 "TO_SOT_Packages_SMD:TO-252-3_TabPin4" H 6200 3200 60  0001 C CNN
 F 3 "" H 6200 3200 60  0001 C CNN
 	1    6200 3150
@@
 F 0 "U4" H 6700 4750 50  0000 L CNN
 F 1 "MCP3421A0T-E/CH" H 6300 4850 50  0000 L CNN
-F 2 "" H 7100 4450 50  0001 C CIN
+F 2 "TO_SOT_Packages_SMD:SOT-23-6_Handsoldering" H 7100 4450 50  0001 C CIN
 F 3 "" H 7100 4450 50  0001 C CNN
 	1    7100 4450
@@
 F 0 "IC1" H 9600 2550 50  0000 L CNN
 F 1 "ADC-20-4" H 9600 2450 50  0000 L CNN
-F 2 "ADC-20-4+" H 8950 2800 50  0001 L CNN
+F 2 "rf_noise:ADC-20-4+" H 8950 2800 50  0001 L CNN
 F 3 "https://www.minicircuits.com/pdfs/ADC-20-4.pdf" H 8300 2650 50  0001 L CNN
 F 4 "Surface Mount Directional Coupler" H 8550 1700 50  0001 L CNN "Description"
@@
 F 0 "D2" H 8450 2900 50  0000 C CNN
 F 1 "SMS3922-079LF" V 8450 2300 50  0000 C CNN
-F 2 "" H 8450 2800 50  0001 C CNN
+F 2 "Diodes_SMD:D_SOD-523" H 8450 2800 50  0001 C CNN
 F 3 "" H 8450 2800 50  0001 C CNN
 	1    8450 2800
@@
 $EndComp
 $Comp
-L C_Small C?
+L C_Small C12
 U 1 1 5D5465D6
 P 8450 4600
-F 0 "C?" H 8460 4670 50  0000 L CNN
+F 0 "C12" H 8460 4670 50  0000 L CNN
 F 1 "1nF" V 8300 4550 50  0000 L CNN
 F 2 "Capacitors_SMD:C_0805_HandSoldering" H 8450 4600 50  0001 C CNN
@@
 $EndComp
 $Comp
-L GND #PWR?
+L GND #PWR033
 U 1 1 5D546718
 P 8450 4850
-F 0 "#PWR?" H 8450 4600 50  0001 C CNN
+F 0 "#PWR033" H 8450 4600 50  0001 C CNN
 F 1 "GND" H 8450 4700 50  0000 C CNN
 F 2 "" H 8450 4850 50  0001 C CNN
