File: africube4.sch (KiCad schematic (older format))
At the start: 30 parts, among them J1 SMA Edge FM, J2 Conn_01x04, J3 RPi_GPIO, J4 Conn_01x02, U1 TQP7M9105, U2 SXBP-150+, U3 BA178M05FP-E2

Commit message: updated the pcd file to africube 4 by readding inductor L5
Parts:
- removed C3: 4.7uF 16V, Capacitors_SMD:C_0805_HandSoldering, symbol africube3-rescue:CP_Small-_saved_africube2-cache
- removed D1: LED, LEDs:LED_0805_HandSoldering, symbol africube3-rescue:LED-_saved_africube2-cache
- added C3: 4.7uF, Resistor_SMD:R_0805_2012Metric_Pad1.20x1.40mm_HandSolder, symbol africube3-rescue:C_Small-_saved_africube2-cache
- added D1: LED, Resistor_SMD:R_0805_2012Metric_Pad1.20x1.40mm_HandSolder, symbol Device:LED
- added L5: 0, Inductor_SMD:L_12x12mm_H8mm, symbol africube3-rescue:L-_saved_africube2-cache
- J3: footprint Connector_PinSocket_2.54mm:PinSocket_2x20_P2.54mm_Vertical_SMD -> Connector_PinSocket_2.54mm:PinSocket_2x20_P2.54mm_Vertical
- R1: footprint Resistors_SMD:R_0805_HandSoldering -> Resistor_SMD:R_0805_2012Metric_Pad1.20x1.40mm_HandSolder
Connections:
- wire segments 90 -> 95
Other:
- moved on the sheet: J4
